Commit message: camera

File: src/dofbot_description/urdf/dofbot.gazebo.urdf.xacro (robot description, xacro)
@@ -33,11 +33,11 @@
         <joint>${parent_joint}</joint>
         <mimicJoint>${mimic_joint}</mimicJoint>
-        <xacro:if value="${has_pid}">                     <!-- if set to true, PID parameters from "/gazebo_ros_control/pid_gains/${mimic_joint}" are loaded -->
-          <hasPID />
+        <xacro:if value="${has_pid}">
+        <hasPID />
         </xacro:if>
         <multiplier>${multiplier}</multiplier>
         <offset>${offset}</offset>
-        <sensitiveness>${sensitiveness}</sensitiveness>   <!-- if absolute difference between setpoint and process value is below this threshold, do nothing; 0.0 = disable [rad] -->
-        <maxEffort>${max_effort}</maxEffort>              <!-- only taken into account if has_pid:=true [Nm] -->
+        <sensitiveness>${sensitiveness}</sensitiveness>
+        <maxEffort>${max_effort}</maxEffort>
         <xacro:unless value="${robot_namespace == ''}">
           <robotNamespace>${robot_namespace}</robotNamespace>
@@ -239,6 +239,6 @@
         <material><color rgba="0.7 0.7 0.7 1"/></material>
     </gazebo>
-    <!--xacro:include filename="$(find as_arm_description)/urdf/camera.xacro"/>
-    <xacro:include filename="$(find as_arm_description)/urdf/camera_y.xacro"/>
+    <xacro:include filename="$(find dofbot_description)/urdf/camera.xacro"/>
+    <!--xacro:include filename="$(find as_arm_description)/urdf/camera_y.xacro"/>
     <xacro:include filename="$(find as_arm_description)/urdf/sink.xacro"/-->
     <joint name="wrist_rot_joint" type="revolute">
@@ -306,4 +306,7 @@
         <mimic joint="gripper_joint" multiplier="-1" offset="0" />
     </joint>
+    <xacro:mimic_joint_plugin_gazebo name_prefix="rlink_joint2"
+    parent_joint="gripper_joint" mimic_joint="rlink_joint2"
+    has_pid="false" multiplier="-1.0" max_effort="10.0" />
     <link name="rlink3">
         <visual>
@@ -332,5 +335,8 @@
         <mimic joint="gripper_joint" multiplier="1" offset="0" />
     </joint>
-    <!--link name="llink1">
+    <xacro:mimic_joint_plugin_gazebo name_prefix="rlink_joint3"
+    parent_joint="gripper_joint" mimic_joint="rlink_joint3"
+    has_pid="false" multiplier="1.0" max_effort="10.0" />
+    <link name="llink1">
         <visual>
             <origin xyz="0 0 0" rpy="0 0 0"/>
@@ -418,5 +424,5 @@
     <xacro:mimic_joint_plugin_gazebo name_prefix="llink_joint3"
     parent_joint="gripper_joint" mimic_joint="llink_joint3"
-    has_pid="false" multiplier="-1.0" max_effort="10.0" /-->
+    has_pid="false" multiplier="-1.0" max_effort="10.0" />
     <!-- transmission block -->
     <xacro:transmission_block joint_name="arm_joint1"/>
